File: OpenMacro-PCB/OpenMacro-PCB.kicad_pcb (KiCad board)
At the start: 2 copper layers, 100 x 91.8 mm, 15 parts, among them P1 RFID-RC522-MODULE, SW1 SW_Push, SW2 SW_Push, SW3 SW_Push, SW4 SW_Push, SW5 SW_Push, SW6 SW_Push, SW7 SW_Push, SW8 SW_Push, SW9 SW_Push, U1 AMS1117-3.3, U2 Arduino_Micro

Commit message: Update kicad_pcb.
Parts:
- added ?: , , F.Cu at (149.0, 68.0)
- added ?: , , F.Cu at (149.0, 153.0)
- added ?: , , F.Cu at (55.0, 153.0)
- added ?: , , F.Cu at (98.0, 68.0)
- added C1: 1uF, Capacitor_SMD:C_1206_3216Metric_Pad1.33x1.80mm_HandSolder, B.Cu at (89.7, 130.5)
- added C2: 1uF, Capacitor_SMD:C_1206_3216Metric_Pad1.33x1.80mm_HandSolder, B.Cu at (83.2, 130.6)
- added G***: LOGO, images:dog5, F.Cu at (124.3, 82.5)
- added G***: LOGO, images:rick_roll, B.Cu at (123.0, 84.6)
- added G***: LOGO, images:dog5, B.Cu at (81.2, 69.4)
- added G***: LOGO, images:dog2, B.Cu at (100.3, 75.9)
- added G***: LOGO, images:rick_qr, B.Cu at (93.0, 88.5)
- added G***: LOGO, images:dog1, B.Cu at (89.4, 116.6)
- added G***: LOGO, images:dog4, B.Cu at (112.2, 151.8)
- added G***: LOGO, images:dog5, B.Cu at (120.5, 70.5)
- added G***: LOGO, images:dog4f, B.Cu at (145.7, 71.8)
- added G***: LOGO, images:dog1, B.Cu at (62.5, 153.0)
- added G***: LOGO, images:dog7, F.Cu at (148.8, 81.9)
- added G***: LOGO, images:dog4f, F.Cu at (131.0, 91.6)
- added G***: LOGO, images:dog5, F.Cu at (54.0, 134.5)
- added G***: LOGO, images:dog5, F.Cu at (81.8, 106.8)
- added G***: LOGO, images:dog4, F.Cu at (86.1, 128.2)
- added G***: LOGO, images:dog1, F.Cu at (87.5, 153.0)
- added G***: LOGO, images:dog3, B.Cu at (131.5, 151.9)
- added G***: LOGO, images:dog7, B.Cu at (63.3, 123.5)
- added J1: I2C_Expand, Connector_PinSocket_2.54mm:PinSocket_1x04_P2.54mm_Horizontal, F.Cu at (91.7, 75.1)
- added R1: 10k, Resistor_SMD:R_1206_3216Metric_Pad1.30x1.75mm_HandSolder, B.Cu at (107.6, 72.1)
- added R2: 10k, Resistor_SMD:R_1206_3216Metric_Pad1.30x1.75mm_HandSolder, B.Cu at (114.0, 72.1)
- added U3: Kaise_Arduino_Micro, Audio_Module:Kaise_Arduino_Micro, F.Cu at (62.0, 59.3)
- ENC1: footprint Rotary_Encoder:RotaryEncoder_Alps_EC11E-Switch_Vertical_H20mm -> Rotary_Encoder:RotaryEncoder_Alps_EC11E-Switch_Vertical_H20mm_CircularMountingHoles
- S1: value RKJXV122400R -> Joystick
- U1: moved to B.Cu
- moved U1 80.9 mm to (88.2, 122.5), turned to 180 degrees
- moved S1 15.7 mm to (64.5, 141.0), turned to 180 degrees
- moved ENC1 1.63 mm to (130.7, 78.0)
- moved Brd1 1.23 mm to (108.8, 78.7)
- moved U2 1.12 mm to (78.4, 110.0)
- moved P1 0.56 mm to (72.2, 125.2)
Connections:
- Brd1 pad 1: unconnected-(Brd1-Pad1) -> GND
- Brd1 pad 2: unconnected-(Brd1-Pad2) -> +5V
- Brd1 pad 3: unconnected-(Brd1-Pad3) -> SCL
- Brd1 pad 4: unconnected-(Brd1-Pad4) -> SDA
- ENC1 pad A: unconnected-(ENC1-PadA) -> D7
- ENC1 pad B: unconnected-(ENC1-PadB) -> D12
- ENC1 pad C: unconnected-(ENC1-PadC) -> GND
- ENC1 pad MP: (no net) -> GND
- ENC1 pad S1: unconnected-(ENC1-PadS1) -> A4
- ENC1 pad S2: unconnected-(ENC1-PadS2) -> GND
- P1 pad 1: unconnected-(P1-Pad1) -> D10
- P1 pad 2: unconnected-(P1-Pad2) -> SCK
- P1 pad 3: unconnected-(P1-Pad3) -> MOSI
- P1 pad 4: unconnected-(P1-Pad4) -> MISO
- P1 pad 6: unconnected-(P1-Pad6) -> GND
- P1 pad 7: unconnected-(P1-Pad7) -> RST
- P1 pad 8: unconnected-(P1-Pad8) -> +3V3
- S1 pad A1: unconnected-(S1-PadA1) -> A2
- S1 pad A11: unconnected-(S1-PadA11) -> +5V
- S1 pad A12: unconnected-(S1-PadA12) -> A3
- S1 pad A13: unconnected-(S1-PadA13) -> GND
- S1 pad B1: unconnected-(S1-PadB1) -> GND
- S1 pad B11: unconnected-(S1-PadB11) -> +5V
- S1 pad B12: unconnected-(S1-PadB12) -> A5
- S1 pad B13: unconnected-(S1-PadB13) -> GND
- S1 pad C1: unconnected-(S1-PadC1) -> A2
- S1 pad D1: unconnected-(S1-PadD1) -> GND
- S1 pad MH1: unconnected-(S1-PadMH1) -> GND
- S1 pad MH2: unconnected-(S1-PadMH2) -> GND
- S1 pad MH3: unconnected-(S1-PadMH3) -> GND
- S1 pad MH4: unconnected-(S1-PadMH4) -> GND
- S1 pad MH5: unconnected-(S1-PadMH5) -> GND
- S1 pad MH6: unconnected-(S1-PadMH6) -> GND
- SW1 pad 1: unconnected-(SW1-Pad1) -> D9
- SW1 pad 2: unconnected-(SW1-Pad2) -> GND
- SW2 pad 1: unconnected-(SW2-Pad1) -> D8
- SW2 pad 2: unconnected-(SW2-Pad2) -> GND
- SW3 pad 1: unconnected-(SW3-Pad1) -> D6
- SW3 pad 2: unconnected-(SW3-Pad2) -> GND
- SW4 pad 1: unconnected-(SW4-Pad1) -> D5
- SW4 pad 2: unconnected-(SW4-Pad2) -> GND
- SW5 pad 1: unconnected-(SW5-Pad1) -> D4
- SW5 pad 2: unconnected-(SW5-Pad2) -> GND
- SW6 pad 1: unconnected-(SW6-Pad1) -> A0
- SW6 pad 2: unconnected-(SW6-Pad2) -> GND
- SW7 pad 1: unconnected-(SW7-Pad1) -> A1
- SW7 pad 2: unconnected-(SW7-Pad2) -> GND
- SW8 pad 1: unconnected-(SW8-Pad1) -> D13
- SW8 pad 2: unconnected-(SW8-Pad2) -> GND
- SW9 pad 1: unconnected-(SW9-Pad1) -> D11
- SW9 pad 2: unconnected-(SW9-Pad2) -> GND
- U1 pad 1: unconnected-(U1-Pad1) -> GND
- U1 pad 2: unconnected-(U1-Pad2) -> +3V3
- U1 pad 3: unconnected-(U1-Pad3) -> +5V
- U2 pad 1: unconnected-(U2-Pad1) -> MOSI
- U2 pad 10: unconnected-(U2-Pad10) -> D5
- U2 pad 11: unconnected-(U2-Pad11) -> D6
- U2 pad 12: unconnected-(U2-Pad12) -> D7
- U2 pad 13: unconnected-(U2-Pad13) -> D8
- U2 pad 14: unconnected-(U2-Pad14) -> D9
- U2 pad 15: unconnected-(U2-Pad15) -> D10
- U2 pad 16: unconnected-(U2-Pad16) -> D11
- U2 pad 17: unconnected-(U2-Pad17) -> D12
- U2 pad 18: unconnected-(U2-Pad18) -> D13
- U2 pad 21: unconnected-(U2-Pad21) -> A0
- U2 pad 22: unconnected-(U2-Pad22) -> A1
- U2 pad 23: unconnected-(U2-Pad23) -> A2
- U2 pad 24: unconnected-(U2-Pad24) -> A3
- U2 pad 25: unconnected-(U2-Pad25) -> A4
- U2 pad 26: unconnected-(U2-Pad26) -> A5
- U2 pad 29: unconnected-(U2-Pad29) -> +5V
- U2 pad 30: unconnected-(U2-Pad30) -> RST
- U2 pad 31: unconnected-(U2-Pad31) -> GND
- U2 pad 33: unconnected-(U2-Pad33) -> MISO
- U2 pad 34: unconnected-(U2-Pad34) -> SCK
- U2 pad 5: unconnected-(U2-Pad5) -> RST
- U2 pad 6: unconnected-(U2-Pad6) -> GND
- U2 pad 7: unconnected-(U2-Pad7) -> SDA
- U2 pad 8: unconnected-(U2-Pad8) -> SCL
- U2 pad 9: unconnected-(U2-Pad9) -> D4
Routing:
- net +5V: track 0.00 -> 216.9 mm, vias 0 -> 3
- net D11: track 0.00 -> 144.4 mm, vias 0 -> 3
- net A0: track 0.00 -> 136.1 mm, vias 0 -> 1
- net D6: track 0.00 -> 117.0 mm, vias 0 -> 2
- net D13: track 0.00 -> 116.6 mm, vias 0 -> 1
- net D8: track 0.00 -> 113.6 mm, vias 0 -> 3
- net SDA: track 0.00 -> 109.0 mm
- net D4: track 0.00 -> 104.7 mm, vias 0 -> 2
- net D12: track 0.00 -> 104.5 mm, vias 0 -> 2
- net SCL: track 0.00 -> 97.8 mm, vias 0 -> 1
- net D9: track 0.00 -> 97.2 mm, vias 0 -> 3
- net D7: track 0.00 -> 97.1 mm, vias 0 -> 2
- net RST: track 0.00 -> 95.3 mm, vias 0 -> 2
- net A1: track 0.00 -> 89.9 mm, vias 0 -> 2
- net A4: track 0.00 -> 88.8 mm, vias 0 -> 1
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- added copper zone on B.Cu, net GND
Other:
- board size 100 x 91.8 mm -> 100 x 91 mm
- board text added: "1U MX-Alps-Choc switches"
- board text added: "5V"
- board text added: "5V I/O"
- board text added: "AMS1117-3.3"
- board text added: "ARDUINO MICRO"
- board text added: "Alps Joystick"
- board text added: "EXPANSION"
- board text added: "Encoder"
- board text added: "GND"
- board text added: "I2C"
- board text added: "JLCJLCJLCJLC"
- board text added: "KAISE MICRO"
- board text added: "OpenMacro PCB Rev.1 by PC & JC"
- board text added: "Rotary"
- board text added: "SCL"
- board text added: "SDA"
- board text added: "SSD1306 Display"
- board text removed: "Display"

Commit message: Serial receive working. Macros still have problems
Parts:
- removed the G*** at (123.0, 84.6)
- removed the G*** at (120.5, 70.5)
- added G***: LOGO, images:rick_pixel, B.Cu at (116.6, 86.1)
- added G***: LOGO, images:dog6f, B.Cu at (121.6, 73.1)
- added G***: LOGO, images:sans_small, B.Cu at (58.9, 68.4)
- added G***: LOGO, images:dog1f, B.Cu at (62.3, 152.0)
- added G***: LOGO, images:dog2f, B.Cu at (112.1, 116.3)
- G***: moved to F.Cu
- moved G*** 42.2 mm to (70.4, 111.5), turned to 0 degrees
- moved G*** 28.8 mm to (128.8, 95.0), turned to 140 degrees
- moved G*** 2.55 mm to (88.4, 129.3)
- moved G*** 2.45 mm to (97.9, 76.4)
- moved G*** 2.43 mm to (90.6, 88.9)
Other:
- board text added: "Expansion"
- board text removed: "EXPANSION"

Commit message: Fix bug in PCB.
Connections:
- Brd1 pad 1: GND -> +5V
- Brd1 pad 2: +5V -> GND
Routing:
- net +5V: track 216.9 -> 212.6 mm
Changed lines of the file:
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@@
     (fp_line (start -12.978 7.595) (end -12.978 -9.005) (layer "F.SilkS") (width 0.12))
     (pad "1" thru_hole oval locked (at -3.62 -10.6 90) (size 2 1.6) (drill 1) (layers *.Cu *.Mask)
-      (net 1 "GND") (pinfunction "GND") (pintype "input"))
+      (net 2 "+5V") (pinfunction "GND") (pintype "input"))
     (pad "2" thru_hole oval locked (at -1.08 -10.6 90) (size 2 1.6) (drill 1) (layers *.Cu *.Mask)
-      (net 2 "+5V") (pinfunction "VCC") (pintype "input"))
+      (net 1 "GND") (pinfunction "VCC") (pintype "input"))
     (pad "3" thru_hole oval locked (at 1.46 -10.6 90) (size 2 1.6) (drill 1) (layers *.Cu *.Mask)
       (net 3 "SCL") (pinfunction "SCL") (pintype "input"))
@@
   (via (at 91.3 133.2) (size 0.9) (drill 0.3) (layers "F.Cu" "B.Cu") (net 2))
   (segment (start 72.4 106.1) (end 73.9 107.6) (width 0.5) (layer "B.Cu") (net 2))
-  (segment (start 107.67 70.48) (end 107.67 68.05) (width 0.3) (layer "B.Cu") (net 2))
+  (segment (start 106.05 72.1) (end 105.13 71.18) (width 0.3) (layer "B.Cu") (net 2))
   (segment (start 73.9 107.6) (end 73.9 109.2) (width 0.5) (layer "B.Cu") (net 2))
   (segment (start 93.6 123.7) (end 92.5 124.8) (width 0.5) (layer "B.Cu") (net 2))
@@
   (segment (start 106.05 72.7) (end 107.95 74.6) (width 0.3) (layer "B.Cu") (net 2))
   (segment (start 73.9 109.2) (end 81.5 116.8) (width 0.5) (layer "B.Cu") (net 2))
+  (segment (start 105.13 71.18) (end 105.13 68.05) (width 0.3) (layer "B.Cu") (net 2))
   (segment (start 91.65 75.1) (end 92.1 75.55) (width 0.5) (layer "B.Cu") (net 2))
   (segment (start 92.5 124.8) (end 91.35 124.8) (width 0.5) (layer "B.Cu") (net 2))
+  (segment (start 101.95 68.05) (end 105.13 68.05) (width 0.5) (layer "B.Cu") (net 2))
   (segment (start 88.95 77.8) (end 91.65 75.1) (width 0.5) (layer "B.Cu") (net 2))
   (segment (start 107.95 74.6) (end 110.55 74.6) (width 0.3) (layer "B.Cu") (net 2))
-  (segment (start 105.91952 66.29952) (end 107.67 68.05) (width 0.5) (layer "B.Cu") (net 2))
   (segment (start 81.5 116.8) (end 91.6 116.8) (width 0.5) (layer "B.Cu") (net 2))
-  (segment (start 106.05 72.1) (end 107.67 70.48) (width 0.3) (layer "B.Cu") (net 2))
   (segment (start 91.3 133.2) (end 91.3 130.5375) (width 0.3) (layer "B.Cu") (net 2))
   (segment (start 91.6 116.8) (end 92.1 117.3) (width 0.5) (layer "B.Cu") (net 2))
+  (segment (start 95 75) (end 101.95 68.05) (width 0.5) (layer "B.Cu") (net 2))
   (segment (start 92.1 117.3) (end 93.6 118.8) (width 0.5) (layer "B.Cu") (net 2))
   (segment (start 110.55 74.6) (end 112.45 72.7) (width 0.3) (layer "B.Cu") (net 2))
-  (segment (start 95 75) (end 103.70048 66.29952) (width 0.5) (layer "B.Cu") (net 2))
   (segment (start 91.3 130.5375) (end 91.2625 130.5) (width 0.3) (layer "B.Cu") (net 2))
   (segment (start 93.6 118.8) (end 93.6 123.7) (width 0.5) (layer "B.Cu") (net 2))
-  (segment (start 103.70048 66.29952) (end 105.91952 66.29952) (width 0.5) (layer "B.Cu") (net 2))
   (segment (start 91.35 130.4125) (end 91.2625 130.5) (width 0.3) (layer "B.Cu") (net 2))
   (segment (start 92.25 75) (end 95 75) (width 0.5) (layer "B.Cu") (net 2))
